File: ADA400A.kicad_sch (KiCad schematic)
At the start: 95 parts, among them J1 BNC, J2 COAX CABLE, K1 TF2E-5V, Q1 NJFET, Q2 NJFET, Q3 Q_NPN_BCE, SW1 MSSA2350G, SW2 MSS-2250G, SW3 MSSA4450G, SW4 MSSA4450G, U1 LT1021-5, U2 INA111, U3 OP27, U4 AD829, U5 LT1021-5, U6 TL072

Commit message: Improve Schematic Accuracy
With thanks to Thorsten Gartner, for pointing out errors in the schematic.
Parts:
- added C19, C20, C21: 47nF 25V, symbol Device:C_Polarized_US
- added C22, C23, C24, C25: 100nF, symbol Device:C
- C10: value 1uF 50V Film -> 1uF 63V 5%
- C11, C16, C18: value C -> 100nF
- C12: value C -> 27pF
- C13: value ?nF -> 1.5nF 1200V 5%
- C14: value 0.05uF? -> 50nF
- C15: value 1uF 50V Film -> 1uF 63V 10%
- C17: value 1uF 50V Film? -> 0.47uF 63V 10%
- C2, C7: value CTRIM -> 2.0-18pF; MPN (none) -> BFC280905217
- C3, C6: value CTRIM -> 1.2-3.5pF; MPN (none) -> BFC280905215
- C4: value ?pF -> 1.2pF
- C5: value Mica ?pF -> Mica 10pF
- C9: value Large Mica ?pF -> Mica 1.2nF
- D2, D3, D4, D5: value D -> 1N4152
- Q3: value Q_NPN_BCE -> 2N3904
- R1: value 20.1 -> 200 5%
- R15: value 130 1% -> 100k
- R20: value 1M 1% -> 1.4K 1%
- R29: value 10k 1% -> 100k 1%
- R3, R7: value 100k 0.1% -> 10k 0.1%
- R38: value 56.2 1% -> 5.62k 1%
- RV1: value 2K -> 20K
- RV5: value CM TRIM -> 200
- RV8: value ?K -> 5K
- U4: symbol Amplifier_Operational:LM741 -> Amplifier_Operational:LT1363
Connections:
- net +15V: now also R32.2, U5.2 (IN), C20.1, C23.1
- net +5V: now also C19.1
- net -15V: now also C21.2, C22.2; no longer D3.2 (A)
- net -5VA: now also C24.1
- net GND: now also C12.1, D3.2 (A), D5.2 (A), R33.1, R37.1, R40.1, U5.4 (GND), C19.2, C20.2, C21.1, C22.1, C23.2, C24.2, C25.2; no longer R38.1
- net at R15.1, U2.6: now also SW3.15
- net at R15.2, R19.2: now also SW3.14; no longer SW3.15
- net at U4.5 (NC): no longer RV7.3
- net at U4.8 (VOS): now also RV7.3
- net at R28.1, R31.1: now also U6.6 (-); no longer U6.2 (-)
- net at C18.1, D4.1 (K), R34.2: now also U6.3 (+); no longer U6.5 (+)
- net at D4.2 (A), R31.2: now also U6.7; no longer U6.1
- net at R29.2, R30.2: now also U6.5 (+); no longer U6.3 (+)
- net at R32.1, R33.2: now also U6.2 (-); no longer U6.6 (-)
- net at R36.1: now also U6.1; no longer U6.7
- net at SW3.11, SW3.9: now also R38.1
- net COMP renamed 5 COMP
- net READOUT renamed SCALE_FACTOR_CODING
- net SCALE_FACTOR_CODING: now also C25.1
- no-connect marks 14 -> 16
Other:
- note added: "- Channel Trim"
- note added: "2 more poles unused"
- note added: "To + Channel"
- note removed: "2 more poles unused?"
- note removed: "Can't find any documentation but presumably these lower resistors activate the 0.1X and 0.01X attenuation on some scopes."
- note removed: "Maybe a trace from here to bottom of 925 ohm?"
- note removed: "Not sure how this is connected but it's pretty clear that it's making a 5V reference."
- note removed: "Other channel"
- note removed: "Pot is only on - channel Probably 2K to match 8250 to other channel's 10K"
- moved on the sheet: C14, C15, C16, C17, C5, C6, C7, R15, R41, R43, R44, U6A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
